File: embedded/raspberry-pi/1.0/pihat.brd (EAGLE design)
At the start: 65 x 56 mm, 33 parts, among them J3 DF13-6P-1.25H, Q3 10mHz, U1 DSPIC33EPXXXGP504, U3 24LC1025-I/SM, U4 24LC1025-I/SM, U5 24LC1025-I/SM, U6 24LC1025-I/SM, U7 MCP2562-E/SN, X1 057-040-1

Commit message: Updated with new design
Parts:
- removed H1, H2, H3, H4: MOUNT-HOLE3.2, holes:3,2
- removed J2: (no value), 15pinD:DB9
- removed R1, R4: 2K2, SparkFun-Passives:0603-RES
- added C10: 220mf, SparkFun:EIA7343
- added C9: 220mf 50v, SparkFun:EIA7343
- added D2: B140-13-F, diode2:SMA
- added L2: 33uh, SparkFun:1812
- added M1, M2, M3, M4: MOUNT-HOLE2.8, tdk:2,8
- added U$2: DF13-8P-1.25H, con-hirose-df13:DF13A-8P-1.25H
- added U2: LM2592HVS-5.0, NSC_By_element14_Batch_1.1:TO170P1435X457-5N
- JP1: value M11PTH -> (none); device 15pinD:1X11 -> 15pinD:DB9_MALE
- moved JP1 54.4 mm to (9.53, 30.5), turned to 90 degrees
- moved Q3 37.4 mm to (61.6, 19.7), turned to 270 degrees
- moved C26 36.3 mm to (46.0, 9.53)
- moved C3 35.2 mm to (60.6, 13.0), turned to 180 degrees
- moved C4 32.9 mm to (57.1, 23.2), turned to 90 degrees
- moved J4 27.7 mm to (31.8, 14.6), turned to 90 degrees
- moved U$1 25.9 mm to (31.1, 20.0)
- moved C17 23.9 mm to (45.7, 26.4)
- moved C28 20.8 mm to (58.4, 10.5), turned to 0 degrees
- moved C15 20.4 mm to (57.5, 17.1), turned to 270 degrees
- moved U1 17.7 mm to (47.6, 18.1), turned to 0 degrees
- moved U7 14.0 mm to (21.9, 14.9)
- moved R2 13.8 mm to (55.6, 30.8), turned to 270 degrees
- moved C27 10.6 mm to (25.1, 19.4)
- moved J3 9.44 mm to (59.7, 33.3)
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Connections:
- removed net CE0#: U1.2, X1.24
- removed net CE1#: U1.3, X1.26
- removed net GPIO13: U1.14, X1.33
- removed net GPIO19: U1.43, X1.35
- removed net GPIO5: U1.41, X1.29
- removed net GPIO6: U1.42, X1.31
- removed net ID_SC: R4.1, U1.44, X1.28
- removed net ID_SD: R1.1, U1.1, X1.27
- removed net MISO: U1.34, X1.21
- removed net MOSI: U1.35, X1.19
- removed net N$1: JP1.10, U1.12
- removed net N$2: JP1.9, U1.13
- removed net SCLK: U1.36, X1.23
- new net N$12: D2.C, L2.1, U2.2
- net +12V: now also C9.A, JP1.1, JP1.9, U2.1; no longer J2.1, J2.9
- net 3.3V: no longer R1.2, R4.2
- net 5V: now also C10.A, L2.2, U2.4; no longer JP1.1
- net CANH: now also JP1.4, JP1.7; no longer J2.4, J2.7
- net CANL: now also JP1.2, JP1.8; no longer J2.2, J2.8
- net GND: now also C10.C, C9.C, D2.A, JP1.3, JP1.5, JP1.6, JP1.G1, JP1.G2, U$2.P$8, U2.3, U2.5, U2.6; no longer J2.3, J2.5, J2.6, J2.G1, J2.G2, JP1.11
- net N$3: now also U$2.P$7; no longer JP1.8
- net N$4: now also U$2.P$6; no longer JP1.7
- net N$5: now also U$2.P$5; no longer JP1.6
- net N$6: now also U$2.P$4; no longer JP1.5
- net N$7: now also U$2.P$3; no longer JP1.4
- net N$8: now also U$2.P$2; no longer JP1.3
- net N$9: now also U$2.P$1; no longer JP1.2
Routing:
- net CE1#: track 64.2 -> 0.00 mm, vias 1 -> 0
- net ID_SD: track 62.5 -> 0.00 mm, vias 3 -> 0
- net GPIO19: track 60.8 -> 0.00 mm, vias 1 -> 0
- net ID_SC: track 60.5 -> 0.00 mm, vias 3 -> 0
- net CE0#: track 59.4 -> 0.00 mm, vias 1 -> 0
- net GPIO6: track 56.3 -> 0.00 mm, vias 1 -> 0
- net GPIO5: track 51.0 -> 0.00 mm, vias 1 -> 0
- net GND: track 45.7 -> 1.27 mm, vias 30 -> 1
- net 5V: track 91.6 -> 48.5 mm, vias 4 -> 0
- net 3.3V: track 0.00 -> 42.9 mm, vias 0 -> 23
- net SCLK: track 41.6 -> 0.00 mm, vias 1 -> 0
- net N$9: track 48.7 -> 13.9 mm, vias 2 -> 0
- net MOSI: track 33.4 -> 0.00 mm, vias 1 -> 0
- net MISO: track 33.3 -> 0.00 mm, vias 1 -> 0
- net GPIO13: track 33.1 -> 0.00 mm
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- added copper zone on layer 16, net 3.3V
- added copper zone on layer 1, net 5V
- added copper zone on layer 1, net GND
- removed copper zone on layer 1, net 3.3V
- removed copper zone on layer 16, net GND
Other:
- outline, holes or cut-outs redrawn
