File: embedded/raspberry-pi/1.0/pihat.sch (EAGLE design)
At the start: 33 parts, among them J3 DF13-6P-1.25H, Q3 10mHz, U1 DSPIC33EPXXXGP504, U3 24LC1025-I/SM, U4 24LC1025-I/SM, U5 24LC1025-I/SM, U6 24LC1025-I/SM, U7 MCP2562-E/SN, X1 057-040-1

Commit message: Updated with new design
Parts:
- removed H1, H2, H3, H4: MOUNT-HOLE3.2, holes:MOUNT-HOLE3.2
- removed J2: (no value), 15pinD:DB9FEMALE
- removed R1, R4: 2K2, SparkFun-Passives:RESISTOR0603-RES
- added C10: 220mf, SparkFun:CAP_POL7343
- added C9: 220mf 50v, SparkFun:CAP_POL7343
- added D2: B140-13-F, diode2:DIODE-SCHOTTKY-SMA
- added L2: 33uh, SparkFun:INDUCTOR
- added M1, M2, M3, M4: MOUNT-HOLE2.8, tdk:MOUNT-HOLE2.8
- added U$2: DF13-8P-1.25H, con-hirose-df13:DF13-8P-1.25H
- added U2: LM2592HVS-5.0, NSC_By_element14_Batch_1.1:LM2592HVS-5.0
- JP1: value M11PTH -> (none); device 15pinD:M11PTH -> 15pinD:DB9MALE
Connections:
- removed net CE0#: U1.RP54/RC6, X1-24.S
- removed net CE1#: U1.RP55/RC7, X1-26.S
- removed net GPIO13: U1.RPI46/T3CK/RB14, X1-33.S
- removed net GPIO19: U1.RP39/INT0/RB7, X1-35.S
- removed net GPIO5: U1.PGED2/ASDA2/RP37/RB5, X1-29.S
- removed net GPIO6: U1.RGEC2/ASCL2/RP38/RB6, X1-31.S
- removed net ID_SC: R4.1, U1.TCK/CVREF10/ASCL1/RP40/T4CK/RB8, X1-28.S
- removed net ID_SD: R1.1, U1.TMS/ASDA1/RP4/RB9, X1-27.S
- removed net MISO: U1.CVREF20/SDO1/RP20/T1CK/RA4, X1-21.S
- removed net MOSI: U1.SDI1/RPI25/RA9, X1-19.S
- removed net N$1: JP1.10, U1.TDO/RA10
- removed net N$2: JP1.9, U1.TDI/RA7
- removed net SCLK: U1.SCK1/RPI51/RC3, X1-23.S
- new net N$12: D2.C, L2.1, U2.OUT
- net +12V: now also C9.+, JP1.1, JP1.9, U2.VIN; no longer J2.1, J2.9
- net 3.3V: no longer R1.2, R4.2
- net 5V: now also C10.+, L2.2, U2.FB; no longer JP1.1
- net CANH: now also JP1.4, JP1.7; no longer J2.4, J2.7
- net CANL: now also JP1.2, JP1.8; no longer J2.2, J2.8
- net GND: now also C10.-, C9.-, D2.A, JP1.3, JP1.5, JP1.6, JP1.SHIELD, U$2.8, U2.GND, U2.GND_2, U2.~ON/OFF; no longer J2.3, J2.5, J2.6, J2.SHIELD, JP1.11
- net N$3: now also U$2.7; no longer JP1.8
- net N$4: now also U$2.6; no longer JP1.7
- net N$5: now also U$2.5; no longer JP1.6
- net N$6: now also U$2.4; no longer JP1.5
- net N$7: now also U$2.3; no longer JP1.4
- net N$8: now also U$2.2; no longer JP1.3
- net N$9: now also U$2.1; no longer JP1.2

Commit message: Updated build to make simplere and comply with pi spec
Parts:
- C10, C9: PARTNO (none) -> T545X227M016ATE035
- D2: PARTNO (none) -> B140-13-F
- JP1: PARTNO (none) -> 5747840-3
- L2: PARTNO (none) -> B78108S1333K
- U$2: PARTNO (none) -> DF13-8P-1.25H(50)
- U2: PARTNO (none) -> LM2592HVSX-5.0/NOPB
Changed lines of the file:
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@@
 <part name="SUPPLY8" library="supply2" deviceset="GND" device=""/>
 <part name="SUPPLY11" library="supply2" deviceset="GND" device=""/>
-<part name="U$2" library="con-hirose-df13" deviceset="DF13-8P-1.25" device="H"/>
+<part name="U$2" library="con-hirose-df13" deviceset="DF13-8P-1.25" device="H">
+<attribute name="PARTNO" value="DF13-8P-1.25H(50)"/>
+</part>
 <part name="SUPPLY14" library="supply2" deviceset="GND" device=""/>
-<part name="C10" library="SparkFun" deviceset="CAP_POL" device="7343" value="220mf"/>
-<part name="C9" library="SparkFun" deviceset="CAP_POL" device="7343" value="220mf 50v"/>
+<part name="C10" library="SparkFun" deviceset="CAP_POL" device="7343" value="220mf">
+<attribute name="PARTNO" value="T545X227M016ATE035"/>
+</part>
+<part name="C9" library="SparkFun" deviceset="CAP_POL" device="7343" value="220mf 50v">
+<attribute name="PARTNO" value="T545X227M016ATE035"/>
+</part>
 <part name="SUPPLY18" library="supply2" deviceset="GND" device=""/>
 <part name="SUPPLY21" library="supply2" deviceset="GND" device=""/>
-<part name="L2" library="SparkFun" deviceset="INDUCTOR" device="" value="33uh"/>
-<part name="D2" library="diode2" deviceset="DIODE-SCHOTTKY-" device="SMA" value="B140-13-F"/>
-<part name="U2" library="NSC_By_element14_Batch_1.1" deviceset="LM2592HVS-5.0" device=""/>
+<part name="L2" library="SparkFun" deviceset="INDUCTOR" device="" value="33uh">
+<attribute name="PARTNO" value="B78108S1333K"/>
+</part>
+<part name="D2" library="diode2" deviceset="DIODE-SCHOTTKY-" device="SMA" value="B140-13-F">
+<attribute name="PARTNO" value="B140-13-F"/>
+</part>
+<part name="U2" library="NSC_By_element14_Batch_1.1" deviceset="LM2592HVS-5.0" device="">
+<attribute name="PARTNO" value="LM2592HVSX-5.0/NOPB"/>
+</part>
 <part name="SUPPLY12" library="SparkFun-Aesthetics" deviceset="5V" device=""/>
-<part name="JP1" library="15pinD" deviceset="DB9" device="MALE"/>
+<part name="JP1" library="15pinD" deviceset="DB9" device="MALE">
+<attribute name="PARTNO" value="5747840-3"/>
+</part>
 <part name="M1" library="tdk" deviceset="MOUNT-HOLE" device="2.8"/>
 <part name="M2" library="tdk" deviceset="MOUNT-HOLE" device="2.8"/>
@@
 <attribute name="NAME" x="40.64" y="191.135" size="1.778" layer="95" rot="R90"/>
 <attribute name="VALUE" x="43.815" y="196.5325" size="1.778" layer="96"/>
+<attribute name="PARTNO" x="50.8" y="193.04" size="1.778" layer="96" display="off"/>
 </instance>
 <instance part="SUPPLY14" gate="GND" x="254" y="147.32"/>
-<instance part="C10" gate="G$1" x="233.68" y="190.5"/>
-<instance part="C9" gate="G$1" x="149.86" y="203.2"/>
+<instance part="C10" gate="G$1" x="233.68" y="190.5">
+<attribute name="PARTNO" x="233.68" y="190.5" size="1.778" layer="96" display="off"/>
+</instance>
+<instance part="C9" gate="G$1" x="149.86" y="203.2">
+<attribute name="PARTNO" x="149.86" y="203.2" size="1.778" layer="96" display="off"/>
+</instance>
 <instance part="SUPPLY18" gate="GND" x="160.02" y="182.88" rot="MR0"/>
 <instance part="SUPPLY21" gate="GND" x="233.68" y="182.88" rot="MR0"/>
@@
 <attribute name="NAME" x="215.9" y="198.12" size="1.778" layer="95"/>
 <attribute name="VALUE" x="226.06" y="198.12" size="1.778" layer="96"/>
+<attribute name="PARTNO" x="223.52" y="195.58" size="1.778" layer="96" display="off"/>
 </instance>
 <instance part="D2" gate="G$1" x="210.82" y="190.5" smashed="yes" rot="R90">
 <attribute name="NAME" x="208.685" y="188.636" size="1.524" layer="95" rot="R90"/>
 <attribute name="VALUE" x="213.901" y="189.77" size="1.524" layer="96"/>
-</instance>
-<instance part="U2" gate="A" x="185.42" y="198.12"/>
+<attribute name="PARTNO" x="210.82" y="190.5" size="1.778" layer="96" display="off"/>
+</instance>
+<instance part="U2" gate="A" x="185.42" y="198.12">
+<attribute name="PARTNO" x="185.42" y="198.12" size="1.778" layer="96" display="off"/>
+</instance>
 <instance part="SUPPLY12" gate="G$1" x="233.68" y="210.82"/>
-<instance part="JP1" gate="G$1" x="264.16" y="162.56"/>
+<instance part="JP1" gate="G$1" x="264.16" y="162.56">
+<attribute name="PARTNO" x="264.16" y="162.56" size="1.778" layer="96" display="off"/>
+</instance>
 <instance part="M1" gate="G$1" x="193.04" y="60.96" smashed="yes">
 <attribute name="NAME" x="196.85" y="60.96" size="1.27" layer="95"/>
